Commit message: four

File: catkin_ws/src/turtlebot3/turtlebot3_description/urdf/turtlebot3_waffle_pi.urdf.xacro (robot description, xacro)
@@ -186,5 +186,5 @@
   <link name="camera_rgb_optical_frame"/>
 <joint name="light_sensor_joint" type="fixed">
-    <origin xyz="0.08 -0.07 0.1" rpy="0.0 1.57 0"/>
+    <origin xyz="0.08 -0.07 0.1" rpy="0.0 1.3 0"/>
     <parent link="base_link"/>
     <child link="light_sensor__link"/>
@@ -210,5 +210,5 @@
 </link>
 <joint name="light_sensor_joint_left" type="fixed">
-  <origin xyz="0.08 0.07 0.1" rpy="0.0 1.57 0"/>
+  <origin xyz="0.08 0.07 0.1" rpy="0.0 1.3 0"/>
   <parent link="base_link"/>
   <child link="light_sensor__link_left"/>
